File: Diseno_1/Diseno_1.sch (KiCad schematic (older format))
At the start: 1 part, among them U21 TPS563201

Commit message: s
Parts:
- removed U21: TPS563201, ZYNQ_7000:TPS563201, symbol Zynq_7000:TPS563201
- added U1: XC7Z010-BUENO, ZYNQ_7000:BGA-400_20x20_17.0x17.0mm, symbol Zynq_7000:XC7Z010-BUENO
Connections:
- net labels added: GND
- net labels removed: XC7Z010
- wire segments 8 -> 12
Changed lines of the file:
@@
 EESchema Schematic File Version 4
-LIBS:Diseno_1-cache
 EELAYER 30 0
 EELAYER END
@@
 $EndDescr
 $Comp
-L Zynq_7000:XC7Z010 #ZYNQ_07000101
-U 5 1 5FE18120
-P 6100 3550
-F 0 "#ZYNQ_07000101" H 6125 6057 50  0000 C CNN
-F 1 "XC7Z010" H 5800 1100 50  0001 C CNN
-F 2 "ZYNQ_7000:BGA-400_20x20_17.0x17.0mm" H 5950 1100 50  0001 C CNN
-F 3 "" H 5950 1100 50  0001 C CNN
-	5    6100 3550
+L Zynq_7000:XC7Z010-BUENO U1
+U 1 1 5FF23D7A
+P 5150 3350
+F 0 "U1" H 5175 4398 50  0000 C CNN
+F 1 "XC7Z010-BUENO" H 5175 4307 50  0000 C CNN
+F 2 "ZYNQ_7000:BGA-400_20x20_17.0x17.0mm" H 5050 100 50  0001 C CNN
+F 3 "" H 5050 100 50  0001 C CNN
+	1    5150 3350
 	1    0    0    -1
 $EndComp
 $Comp
-L Zynq_7000:TPS563201 U21
-U 1 1 5FDFEF21
-P 9150 2750
-F 0 "U21" H 9125 3231 50  0000 C CNN
-F 1 "TPS563201" H 9125 3140 50  0000 C CNN
-F 2 "ZYNQ_7000:TPS563201" H 8800 3000 50  0001 C CNN
-F 3 "https://www.ti.com/lit/ds/symlink/tps563201.pdf?ts=1608479868872&ref_url=https%253A%252F%252Fwww.google.com%252F" H 8800 3000 50  0001 C CNN
-	1    9150 2750
+L power:GND #PWR0101
+U 1 1 5FF2901C
+P 5800 4400
+F 0 "#PWR0101" H 5800 4150 50  0001 C CNN
+F 1 "GND" H 5805 4227 50  0000 C CNN
+F 2 "" H 5800 4400 50  0001 C CNN
+F 3 "" H 5800 4400 50  0001 C CNN
+	1    5800 4400
 	1    0    0    -1
 $EndComp
 Wire Wire Line
-	8650 2600 7150 2600
+	5800 4000 5750 4000
 Wire Wire Line
-	7150 2600 7150 2550
+	5750 4000 5750 3800
+Connection ~ 5750 4000
+Connection ~ 5750 2750
 Wire Wire Line
-	8650 2850 8650 4550
+	5750 2750 5750 2650
+Connection ~ 5750 2850
 Wire Wire Line
-	8650 4550 7150 4550
+	5750 2850 5750 2750
+Connection ~ 5750 2950
 Wire Wire Line
-	7150 4550 7150 4450
+	5750 2950 5750 2850
+Connection ~ 5750 3200
 Wire Wire Line
-	9550 2700 9550 2600
+	5750 3200 5750 2950
+Connection ~ 5750 3300
 Wire Wire Line
-	9550 2600 9600 2600
+	5750 3300 5750 3200
+Connection ~ 5750 3400
 Wire Wire Line
-	9600 2850 9600 2600
-Connection ~ 9600 2600
+	5750 3400 5750 3300
+Connection ~ 5750 3600
+Wire Wire Line
+	5750 3600 5750 3400
+Connection ~ 5750 3700
+Wire Wire Line
+	5750 3700 5750 3600
+Connection ~ 5750 3800
+Wire Wire Line
+	5750 3800 5750 3700
+Wire Wire Line
+	5800 4000 5800 4400
 $EndSCHEMATC

Commit message: d
Parts:
- removed U1: XC7Z010-BUENO, ZYNQ_7000:BGA-400_20x20_17.0x17.0mm, symbol Zynq_7000:XC7Z010-BUENO
- added C1, C3, C4, C5, C7, C8, C? (x6): 10uF, Capacitor_SMD:C_0805_2012Metric, symbol Device:C
- added C2, C6, C? (x2): 100nF, Capacitor_SMD:C_0805_2012Metric, symbol Device:C
- added L1, L2, L? (x2): 4.7uH, Inductor_SMD:L_0805_2012Metric, symbol Device:L
- added Q1, Q2, Q? (x2): MMBT3904, Package_TO_SOT_SMD:SOT-23, symbol Transistor_BJT:MMBT3904
- added R1, R4, R5, R? (x3): 10k, Resistor_SMD:R_0805_2012Metric, symbol Device:R
- added R2, R?: 33k, Resistor_SMD:R_0805_2012Metric, symbol Device:R
- added R3, R6, R? (x2): 100k, Resistor_SMD:R_0805_2012Metric, symbol Device:R
- added R7: 75k, Resistor_SMD:R_0805_2012Metric, symbol Device:R
- added R? (x3): 0R, Resistor_SMD:R_0805_2012Metric, symbol Device:R
- added R?: 79k, Resistor_SMD:R_0805_2012Metric, symbol Device:R
- added U1, U2, U? (x2): TPS563201, ZYNQ_7000:TPS563201, symbol Zynq_7000:TPS563201
- added U? (x2): XC7Z010-BUENO, ZYNQ_7000:BGA-400_20x20_17.0x17.0mm, symbol Zynq_7000:XC7Z010-BUENO
Connections:
- net GND: now also C1.2, C3.2, C4.2, C5.2, C7.2, C8.2, C?.2, C?.2, C?.2, C?.2, C?.2, C?.2, Q1.2 (E), Q2.2 (E), Q?.2 (E), Q?.2 (E), R3.2, R7.2, R?.2, R?.2, U1.1 (GND), U2.1 (GND), U?.1 (GND), U?.1 (GND), U?.A18 (GND_37), U?.A8 (GND_35), U?.B1 (GND_39), U?.B11 (GND_41), U?.C14 (GND_45), U?.C4 (GND_43), U?.C9 (GND_26), U?.D17 (GND_49), U?.E10 (GND_51), U?.E20 (GND_53), U?.F3 (GND_55), U?.F7 (GND_57), U?.G10 (GND_59), U?.G12 (GND_2), U?.G16 (GND_4), U?.H11 (GND_10), U?.H13 (GND_12), U?.H19 (GND_14), U?.H7 (GND_6), U?.H9 (GND_8), U?.J12 (GND_20), U?.J2 (GND_16), U?.J8 (GND_18), U?.K11 (GND_47), U?.K13 (GND_28), U?.K15 (GND_31), U?.K5 (GND_22), U?.K7 (GND_24), U?.L12 (GND_40), U?.L18 (GND_58), U?.L8 (GND_56), U?.M1 (GND_32), U?.M11 (GND_42), U?.M13 (GND_3), U?.M7 (GND_1), U?.N10 (GND_44), U?.N12 (GND_7), U?.N14 (GND_34), U?.N4 (GND_33), U?.N8 (GND_5), U?.P11 (GND_11), U?.P13 (GND_30), U?.P17 (GND_13), U?.P7 (GND_9), U?.P9 (GND_46), U?.R12 (GND_15), U?.R20 (GND_36), U?.R8 (GND_48), U?.T13 (GND_19), U?.T3 (GND_17), U?.T7 (GND_50), U?.U16 (GND_21), U?.U6 (GND_29), U?.V19 (GND_23), U?.V9 (GND_52), U?.W12 (GND_25), U?.W2 (GND_38), U?.Y15 (GND_27), U?.Y5 (GND_54)
- new net: C2.1, L1.1, U2.2 (SW)
- new net: R2.2, R3.1, U2.4 (VFB)
- new net: R1.1, U2.5 (EN)
- new net: C2.2, U2.6 (VBST)
- new net: C6.1, L2.1, U1.2 (SW)
- new net: R6.2, R7.1, U1.4 (VFB)
- new net: Q2.3 (C), R5.1, U1.5 (EN)
- new net: C6.2, U1.6 (VBST)
- new net: Q1.3 (C), Q2.1 (B), R4.1
- new net: C?.1, L?.1, U?.2 (SW) (x2)
- new net: R?.1, R?.2, U?.4 (VFB) (x2)
- new net: R?.1, U?.5 (EN)
- new net: C?.2, U?.6 (VBST) (x2)
- new net: Q?.3 (C), R?.1, U?.5 (EN)
- new net: Q?.1 (B), Q?.3 (C), R?.1
- new net: Q?.1 (B), R?.1
- new net +1V0: C3.1, C4.1, L1.2, Q1.1 (B), R2.1, U?.G11 (VCCBRAM_2), U?.G13 (VCCINT_5), U?.G7 (VCCPINT_6), U?.H10 (VCCBRAM_1), U?.H12 (VCCINT_8), U?.J13 (VCCINT_6), U?.J7 (VCCPINT_3), U?.K12 (VCCINT_7), U?.L13 (VCCINT_1), U?.L7 (VCCPINT_4), U?.M12 (VCCINT_3), U?.N13 (VCCINT_2), U?.N7 (VCCPINT_5), U?.P12 (VCCINT_9), U?.P8 (VCCPINT_1), U?.R13 (VCCINT_4), U?.R7 (VCCPINT_2)
- new net +1V35: C?.1, C?.1, L?.2, R?.1, R?.2, U?.A3 (VCCO_DDR_502_2), U?.D2 (VCCO_DDR_502_1), U?.E5 (VCCO_DDR_502_8), U?.G1 (VCCO_DDR_502_9), U?.H4 (VCCO_DDR_502_3), U?.L3 (VCCO_DDR_502_7), U?.P2 (VCCO_DDR_502_5), U?.R5 (VCCO_DDR_502_6), U?.U1 (VCCO_DDR_502_10), U?.V4 (VCCO_DDR_502_4)
- new net +1V8: C7.1, C8.1, L2.2, R6.1, R?.2, U?.F11 (VCCBATT_0), U?.F8 (VCCPAUX_1), U?.G8 (VCCPLL), U?.G9 (VCCPAUX_5), U?.H8 (VCCPAUX_4), U?.J11 (VCCAUX_6), U?.K8 (VCCPAUX_2), U?.L11 (VCCAUX_3), U?.M8 (VCCPAUX_3), U?.N11 (VCCAUX_2), U?.N9 (VCCAUX_4), U?.P10 (VCCAUX_5), U?.R9 (VCCAUX_1)
- new net +3V3: C?.1, C?.1, L?.2, R?.1, R?.1, R?.1, U?.A13 (VCCO_MIO1_501_4), U?.B16 (VCCO_MIO1_501_2), U?.B6 (VCCO_MIO0_500_1), U?.C19 (VCCO_35_5), U?.D12 (VCCO_MIO1_501_3), U?.D7 (VCCO_MIO0_500_2), U?.E15 (VCCO_MIO1_501_1), U?.F18 (VCCO_35_1), U?.H14 (VCCO_35_6), U?.J17 (VCCO_35_2), U?.K20 (VCCO_35_3), U?.K6 (VCCO_0), U?.M16 (VCCO_35_4), U?.T8 (VCCO_13_3), U?.U11 (VCCO_13_1), U?.W7 (VCCO_13_2), U?.Y10 (VCCO_13_4)
- new net VCC: C1.1, C5.1, C?.1, C?.1, R1.2, R4.2, R5.2, R?.2, R?.2, R?.2, R?.2, U1.3 (IN), U2.3 (IN), U?.3 (IN), U?.3 (IN), U?.N19 (VCCO_34_2), U?.R15 (VCCO_34_1), U?.T18 (VCCO_34_3), U?.V14 (VCCO_13_6), U?.W17 (VCCO_34_5), U?.Y20 (VCCO_34_4)
