File: Diseno_1/Diseno_1.sch (KiCad schematic (older format))
At the start: 0 parts

Commit message: muchas cosas
Changed lines of the file:
@@
 $EndDescr
 $Sheet
-S 3250 4450 1200 850
+S 3000 4150 1750 1400
 U 5FFBC59B
 F0 "Alimentaciones" 50
