File: Diseno_1/ent_sal.sch (KiCad schematic (older format))
At the start: 3 parts, among them U5 XC7Z010-BUENO

Commit message: actualizacion
Connections:
- net BANK34_U13: no longer names the net of JP1.11 (Pin11)
- net BANK34_U13: no longer U5.U13 (IO_L3P_T0_DQS_PUDC_B_34)
- new net GND: U5.U13 (IO_L3P_T0_DQS_PUDC_B_34)
Changed lines of the file:
@@
 Text Label 3350 5700 2    50   ~ 0
 BANK34_U12
-Text Label 3350 5800 2    50   ~ 0
-BANK34_U13
 Text Label 3350 5900 2    50   ~ 0
 BANK34_V13
@@
 	2800 5700 3350 5700
 Wire Wire Line
-	2800 5800 3350 5800
-Wire Wire Line
 	2800 5900 3350 5900
 Wire Wire Line
@@
 Text Label 1800 1750 0    50   ~ 0
 BANK34_U12
-Text Label 1800 1850 0    50   ~ 0
-BANK34_U13
 Text Label 1800 1950 0    50   ~ 0
 BANK34_V13
@@
 Wire Wire Line
 	2350 1750 1800 1750
-Wire Wire Line
-	2350 1850 1800 1850
 Wire Wire Line
 	2350 1950 1800 1950
@@
 Wire Wire Line
 	4950 3800 5500 3800
+$Comp
+L power:GND #PWR0128
+U 1 1 604F949B
+P 3500 5800
+F 0 "#PWR0128" H 3500 5550 50  0001 C CNN
+F 1 "GND" V 3505 5672 50  0000 R CNN
+F 2 "" H 3500 5800 50  0001 C CNN
+F 3 "" H 3500 5800 50  0001 C CNN
+	1    3500 5800
+	0    -1   -1   0
+$EndComp
+Wire Wire Line
+	3500 5800 2800 5800
 $EndSCHEMATC

Commit message: ACT
Parts:
- JP1, JP2: footprint ZYNQ_7000:PINES_50 -> ZYNQ_7000:PINES_50_NUMERO
Changed lines of the file:
@@
 F 0 "JP1" H 2750 4015 50  0000 C CNN
 F 1 "Pines_Bloque_50" H 2750 3924 50  0000 C CNN
-F 2 "ZYNQ_7000:PINES_50" H 2500 3900 50  0001 C CNN
+F 2 "ZYNQ_7000:PINES_50_NUMERO" H 2500 3900 50  0001 C CNN
 F 3 "" H 2500 3900 50  0001 C CNN
 	1    2750 2550
@@
 F 0 "JP2" H 5900 4065 50  0000 C CNN
 F 1 "Pines_Bloque_50" H 5900 3974 50  0000 C CNN
-F 2 "ZYNQ_7000:PINES_50" H 5650 3950 50  0001 C CNN
+F 2 "ZYNQ_7000:PINES_50_NUMERO" H 5650 3950 50  0001 C CNN
 F 3 "" H 5650 3950 50  0001 C CNN
 	1    5900 2600
