File: Diseno_1/Diseno_1.kicad_pcb (KiCad board)
At the start: 2 copper layers, 2 parts

Commit message: s
Parts:
- removed REF**: TPS563201, ZYNQ_7000:TPS563201
- removed REF**: BGA-400_20x20_17.0x17.0mm, ZYNQ_7000:BGA-400_20x20_17.0x17.0mm
- added U1: XC7Z010-BUENO, ZYNQ_7000:BGA-400_20x20_17.0x17.0mm, F.Cu at (275.6, 105.4)
Routing:
- net (no net): track 23.3 -> 0.00 mm
Changed lines of the file:
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@@
     (thickness 1.6)
     (drawings 0)
-    (tracks 4)
+    (tracks 0)
     (zones 0)
-    (modules 2)
-    (nets 1)
+    (modules 1)
+    (nets 11)
   )
   (page A3)
@@
   )
   (net 0 "")
+  (net 1 "Net-(U1-PadM10)")
+  (net 2 "Net-(U1-PadL10)")
+  (net 3 "Net-(U1-PadK10)")
+  (net 4 "Net-(U1-PadJ10)")
+  (net 5 "Net-(U1-PadM9)")
+  (net 6 "Net-(U1-PadL9)")
+  (net 7 "Net-(U1-PadK9)")
+  (net 8 "Net-(U1-PadJ9)")
+  (net 9 "Net-(U1-PadM6)")
+  (net 10 GND)
   (net_class Default "Esta es la clase de red por defecto."
     (clearance 0.2)
@@
     (uvia_dia 0.3)
     (uvia_drill 0.1)
+    (add_net GND)
+    (add_net "Net-(U1-PadJ10)")
+    (add_net "Net-(U1-PadJ9)")
+    (add_net "Net-(U1-PadK10)")
+    (add_net "Net-(U1-PadK9)")
+    (add_net "Net-(U1-PadL10)")
+    (add_net "Net-(U1-PadL9)")
+    (add_net "Net-(U1-PadM10)")
+    (add_net "Net-(U1-PadM6)")
+    (add_net "Net-(U1-PadM9)")
   )
-  (module ZYNQ_7000:TPS563201 (layer F.Cu)
-    (at 185.42 138.43)
-    (fp_text reference REF** (at 12.41044 18.93024) (layer F.SilkS)
+  (module ZYNQ_7000:BGA-400_20x20_17.0x17.0mm (layer F.Cu)
+    (at 275.59 105.41)
+    (attr smd)
+    (fp_text reference U1 (at 0 -9.5) (layer F.SilkS)
       (effects (font (size 1 1) (thickness 0.15)))
     )
-    (fp_text value TPS563201 (at 12.41044 17.93024) (layer F.Fab)
-      (effects (font (size 1 1) (thickness 0.15)))
-    )
-    (pad 6 smd roundrect (at -0.889 1.397) (size 1.1 0.6) (layers F.Cu F.Paste F.Mask) (roundrect_rratio 0.25))
-    (pad 5 smd roundrect (at -1.651 -0.127) (size 1.1 0.6) (layers F.Cu F.Paste F.Mask) (roundrect_rratio 0.25))
-    (pad 4 smd roundrect (at -0.508 -1.778) (size 1.1 0.6) (layers F.Cu F.Paste F.Mask) (roundrect_rratio 0.25))
-    (pad 3 smd roundrect (at 0.254 -3.683) (size 1.1 0.6) (layers F.Cu F.Paste F.Mask) (roundrect_rratio 0.25))
-    (pad 2 smd roundrect (at 2.159 -1.651) (size 1.1 0.6) (layers F.Cu F.Paste F.Mask) (roundrect_rratio 0.25))
-    (pad 1 smd roundrect (at 2.159 -2.54) (size 1.1 0.6) (layers F.Cu F.Paste F.Mask) (roundrect_rratio 0.25))
-  )
-  (module ZYNQ_7000:BGA-400_20x20_17.0x17.0mm (layer F.Cu)
-    (at 165.1 144.78)
-    (attr smd)
-    (fp_text reference REF** (at 0 -9.5) (layer F.SilkS)
-      (effects (font (size 1 1) (thickness 0.15)))
-    )
-    (fp_text value BGA-400_20x20_17.0x17.0mm (at 0 9.5) (layer F.Fab)
+    (fp_text value XC7Z010-BUENO (at 0 9.5) (layer F.Fab)
       (effects (font (size 1 1) (thickness 0.15)))
     )
@@
     (pad U11 smd circle (at 0.4 5.2) (size 0.5 0.5) (layers F.Cu F.Paste F.Mask))
     (pad T11 smd circle (at 0.4 4.4) (size 0.5 0.5) (layers F.Cu F.Paste F.Mask))
-    (pad R11 smd circle (at 0.4 3.6) (size 0.5 0.5) (layers F.Cu F.Paste F.Mask))
+    (pad R11 smd circle (at 0.4 3.6) (size 0.5 0.5) (layers F.Cu F.Paste F.Mask)
+      (net 10 GND))
     (pad P11 smd circle (at 0.4 2.8) (size 0.5 0.5) (layers F.Cu F.Paste F.Mask))
     (pad N11 smd circle (at 0.4 2) (size 0.5 0.5) (layers F.Cu F.Paste F.Mask))
@@
     (pad U10 smd circle (at -0.4 5.2) (size 0.5 0.5) (layers F.Cu F.Paste F.Mask))
     (pad T10 smd circle (at -0.4 4.4) (size 0.5 0.5) (layers F.Cu F.Paste F.Mask))
-    (pad R10 smd circle (at -0.4 3.6) (size 0.5 0.5) (layers F.Cu F.Paste F.Mask))
+    (pad R10 smd circle (at -0.4 3.6) (size 0.5 0.5) (layers F.Cu F.Paste F.Mask)
+      (net 10 GND))
     (pad P10 smd circle (at -0.4 2.8) (size 0.5 0.5) (layers F.Cu F.Paste F.Mask))
     (pad N10 smd circle (at -0.4 2) (size 0.5 0.5) (layers F.Cu F.Paste F.Mask))
-    (pad M10 smd circle (at -0.4 1.2) (size 0.5 0.5) (layers F.Cu F.Paste F.Mask))
-    (pad L10 smd circle (at -0.4 0.4) (size 0.5 0.5) (layers F.Cu F.Paste F.Mask))
-    (pad K10 smd circle (at -0.4 -0.4) (size 0.5 0.5) (layers F.Cu F.Paste F.Mask))
-    (pad J10 smd circle (at -0.4 -1.2) (size 0.5 0.5) (layers F.Cu F.Paste F.Mask))
+    (pad M10 smd circle (at -0.4 1.2) (size 0.5 0.5) (layers F.Cu F.Paste F.Mask)
+      (net 1 "Net-(U1-PadM10)"))
+    (pad L10 smd circle (at -0.4 0.4) (size 0.5 0.5) (layers F.Cu F.Paste F.Mask)
+      (net 2 "Net-(U1-PadL10)"))
+    (pad K10 smd circle (at -0.4 -0.4) (size 0.5 0.5) (layers F.Cu F.Paste F.Mask)
+      (net 3 "Net-(U1-PadK10)"))
+    (pad J10 smd circle (at -0.4 -1.2) (size 0.5 0.5) (layers F.Cu F.Paste F.Mask)
+      (net 4 "Net-(U1-PadJ10)"))
     (pad H10 smd circle (at -0.4 -2) (size 0.5 0.5) (layers F.Cu F.Paste F.Mask))
     (pad G10 smd circle (at -0.4 -2.8) (size 0.5 0.5) (layers F.Cu F.Paste F.Mask))
-    (pad F10 smd circle (at -0.4 -3.6) (size 0.5 0.5) (layers F.Cu F.Paste F.Mask))
+    (pad F10 smd circle (at -0.4 -3.6) (size 0.5 0.5) (layers F.Cu F.Paste F.Mask)
+      (net 10 GND))
     (pad E10 smd circle (at -0.4 -4.4) (size 0.5 0.5) (layers F.Cu F.Paste F.Mask))
     (pad D10 smd circle (at -0.4 -5.2) (size 0.5 0.5) (layers F.Cu F.Paste F.Mask))
@@
     (pad P9 smd circle (at -1.2 2.8) (size 0.5 0.5) (layers F.Cu F.Paste F.Mask))
     (pad N9 smd circle (at -1.2 2) (size 0.5 0.5) (layers F.Cu F.Paste F.Mask))
-    (pad M9 smd circle (at -1.2 1.2) (size 0.5 0.5) (layers F.Cu F.Paste F.Mask))
-    (pad L9 smd circle (at -1.2 0.4) (size 0.5 0.5) (layers F.Cu F.Paste F.Mask))
-    (pad K9 smd circle (at -1.2 -0.4) (size 0.5 0.5) (layers F.Cu F.Paste F.Mask))
-    (pad J9 smd circle (at -1.2 -1.2) (size 0.5 0.5) (layers F.Cu F.Paste F.Mask))
+    (pad M9 smd circle (at -1.2 1.2) (size 0.5 0.5) (layers F.Cu F.Paste F.Mask)
+      (net 5 "Net-(U1-PadM9)"))
+    (pad L9 smd circle (at -1.2 0.4) (size 0.5 0.5) (layers F.Cu F.Paste F.Mask)
+      (net 6 "Net-(U1-PadL9)"))
+    (pad K9 smd circle (at -1.2 -0.4) (size 0.5 0.5) (layers F.Cu F.Paste F.Mask)
+      (net 7 "Net-(U1-PadK9)"))
+    (pad J9 smd circle (at -1.2 -1.2) (size 0.5 0.5) (layers F.Cu F.Paste F.Mask)
+      (net 8 "Net-(U1-PadJ9)"))
     (pad H9 smd circle (at -1.2 -2) (size 0.5 0.5) (layers F.Cu F.Paste F.Mask))
     (pad G9 smd circle (at -1.2 -2.8) (size 0.5 0.5) (layers F.Cu F.Paste F.Mask))
-    (pad F9 smd circle (at -1.2 -3.6) (size 0.5 0.5) (layers F.Cu F.Paste F.Mask))
+    (pad F9 smd circle (at -1.2 -3.6) (size 0.5 0.5) (layers F.Cu F.Paste F.Mask)
+      (net 10 GND))
     (pad E9 smd circle (at -1.2 -4.4) (size 0.5 0.5) (layers F.Cu F.Paste F.Mask))
     (pad D9 smd circle (at -1.2 -5.2) (size 0.5 0.5) (layers F.Cu F.Paste F.Mask))
@@
     (pad V6 smd circle (at -3.6 6) (size 0.5 0.5) (layers F.Cu F.Paste F.Mask))
     (pad U6 smd circle (at -3.6 5.2) (size 0.5 0.5) (layers F.Cu F.Paste F.Mask))
-    (pad T6 smd circle (at -3.6 4.4) (size 0.5 0.5) (layers F.Cu F.Paste F.Mask))
-    (pad R6 smd circle (at -3.6 3.6) (size 0.5 0.5) (layers F.Cu F.Paste F.Mask))
+    (pad T6 smd circle (at -3.6 4.4) (size 0.5 0.5) (layers F.Cu F.Paste F.Mask)
+      (net 10 GND))
+    (pad R6 smd circle (at -3.6 3.6) (size 0.5 0.5) (layers F.Cu F.Paste F.Mask)
+      (net 10 GND))
     (pad P6 smd circle (at -3.6 2.8) (size 0.5 0.5) (layers F.Cu F.Paste F.Mask))
-    (pad N6 smd circle (at -3.6 2) (size 0.5 0.5) (layers F.Cu F.Paste F.Mask))
-    (pad M6 smd circle (at -3.6 1.2) (size 0.5 0.5) (layers F.Cu F.Paste F.Mask))
-    (pad L6 smd circle (at -3.6 0.4) (size 0.5 0.5) (layers F.Cu F.Paste F.Mask))
+    (pad N6 smd circle (at -3.6 2) (size 0.5 0.5) (layers F.Cu F.Paste F.Mask)
+      (net 10 GND))
+    (pad M6 smd circle (at -3.6 1.2) (size 0.5 0.5) (layers F.Cu F.Paste F.Mask)
+      (net 9 "Net-(U1-PadM6)"))
+    (pad L6 smd circle (at -3.6 0.4) (size 0.5 0.5) (layers F.Cu F.Paste F.Mask)
+      (net 10 GND))
     (pad K6 smd circle (at -3.6 -0.4) (size 0.5 0.5) (layers F.Cu F.Paste F.Mask))
-    (pad J6 smd circle (at -3.6 -1.2) (size 0.5 0.5) (layers F.Cu F.Paste F.Mask))
+    (pad J6 smd circle (at -3.6 -1.2) (size 0.5 0.5) (layers F.Cu F.Paste F.Mask)
+      (net 10 GND))
     (pad H6 smd circle (at -3.6 -2) (size 0.5 0.5) (layers F.Cu F.Paste F.Mask))
-    (pad G6 smd circle (at -3.6 -2.8) (size 0.5 0.5) (layers F.Cu F.Paste F.Mask))
-    (pad F6 smd circle (at -3.6 -3.6) (size 0.5 0.5) (layers F.Cu F.Paste F.Mask))
+    (pad G6 smd circle (at -3.6 -2.8) (size 0.5 0.5) (layers F.Cu F.Paste F.Mask)
+      (net 10 GND))
+    (pad F6 smd circle (at -3.6 -3.6) (size 0.5 0.5) (layers F.Cu F.Paste F.Mask)
+      (net 10 GND))
     (pad E6 smd circle (at -3.6 -4.4) (size 0.5 0.5) (layers F.Cu F.Paste F.Mask))
     (pad D6 smd circle (at -3.6 -5.2) (size 0.5 0.5) (layers F.Cu F.Paste F.Mask))
@@
     (pad A1 smd circle (at -7.6 -7.6) (size 0.5 0.5) (layers F.Cu F.Paste F.Mask))
   )
-  (segment (start 173.177 138.303) (end 172.7 138.78) (width 0.25) (layer F.Cu) (net 0))
-  (segment (start 183.769 138.303) (end 173.177 138.303) (width 0.25) (layer F.Cu) (net 0))
-  (segment (start 173.253 139.827) (end 172.7 140.38) (width 0.25) (layer F.Cu) (net 0))
-  (segment (start 184.531 139.827) (end 173.253 139.827) (width 0.25) (layer F.Cu) (net 0))
 )

Commit message: d
Parts:
- added C1: 10uF, Capacitor_SMD:C_0805_2012Metric, F.Cu at (322.2, 105.4)
- added C2: 100nF, Capacitor_SMD:C_0805_2012Metric, F.Cu at (328.0, 100.3)
- added C3: 10uF, Capacitor_SMD:C_0805_2012Metric, F.Cu at (336.6, 97.8)
- added C4: 10uF, Capacitor_SMD:C_0805_2012Metric, F.Cu at (332.7, 97.8)
- added C5: 10uF, Capacitor_SMD:C_0805_2012Metric, F.Cu at (326.8, 105.2)
- added C6: 100nF, Capacitor_SMD:C_0805_2012Metric, F.Cu at (331.3, 100.8)
- added C7: 10uF, Capacitor_SMD:C_0805_2012Metric, F.Cu at (336.8, 96.2)
- added C8: 10uF, Capacitor_SMD:C_0805_2012Metric, F.Cu at (331.2, 105.2)
- added L1: 4.7uH, Inductor_SMD:L_0805_2012Metric, F.Cu at (336.6, 102.9)
- added L2: 4.7uH, Inductor_SMD:L_0805_2012Metric, F.Cu at (336.8, 99.2)
- added Q1: MMBT3904, Package_TO_SOT_SMD:SOT-23, F.Cu at (326.8, 101.4)
- added Q2: MMBT3904, Package_TO_SOT_SMD:SOT-23, F.Cu at (332.4, 97.0)
- added R1: 10k, Resistor_SMD:R_0805_2012Metric, F.Cu at (332.7, 114.3)
- added R2: 33k, Resistor_SMD:R_0805_2012Metric, F.Cu at (344.2, 106.7)
- added R3: 100k, Resistor_SMD:R_0805_2012Metric, F.Cu at (344.2, 101.6)
- added R4: 10k, Resistor_SMD:R_0805_2012Metric, F.Cu at (341.2, 96.2)
- added R5: 10k, Resistor_SMD:R_0805_2012Metric, F.Cu at (335.7, 102.1)
- added R6: 100k, Resistor_SMD:R_0805_2012Metric, F.Cu at (335.6, 105.1)
- added R7: 75k, Resistor_SMD:R_0805_2012Metric, F.Cu at (341.2, 99.2)
- added U2: TPS563201, ZYNQ_7000:TPS563201, F.Cu at (332.7, 105.4)
- U1: value XC7Z010-BUENO -> TPS563201; footprint ZYNQ_7000:BGA-400_20x20_17.0x17.0mm -> ZYNQ_7000:TPS563201
- moved U1 52.6 mm to (327.5, 97.0)

Commit message: s
Parts:
- added C10: 10uF, Capacitor_SMD:C_0805_2012Metric, F.Cu at (111.9, 102.5)
- added C11: 10uF, Capacitor_SMD:C_0805_2012Metric, F.Cu at (75.5, 125.6)
- added C12: 10uF, Capacitor_SMD:C_0805_2012Metric, F.Cu at (80.0, 119.8)
- added C13: 10uF, Capacitor_SMD:C_0805_2012Metric, F.Cu at (90.0, 112.2)
- added C14: 10uF, Capacitor_SMD:C_0805_2012Metric, F.Cu at (85.5, 116.8)
- added C15: 10uF, Capacitor_SMD:C_0805_2012Metric, F.Cu at (81.1, 113.8)
- added C16: 10uF, Capacitor_SMD:C_0805_2012Metric, F.Cu at (111.9, 105.4)
- added C17: 100nF, Capacitor_SMD:C_0805_2012Metric, F.Cu at (86.4, 97.8)
- added C18: 100nF, Capacitor_SMD:C_0805_2012Metric, F.Cu at (86.4, 100.7)
- added C19: 100nF, Capacitor_SMD:C_0805_2012Metric, F.Cu at (90.8, 97.8)
- added C20: 100nF, Capacitor_SMD:C_0805_2012Metric, F.Cu at (106.7, 54.6)
- added C21: 100nF, Capacitor_SMD:C_0805_2012Metric, F.Cu at (97.9, 54.6)
- added C22: 100nF, Capacitor_SMD:C_0805_2012Metric, F.Cu at (102.3, 51.7)
- added C23: 100nF, Capacitor_SMD:C_0805_2012Metric, F.Cu at (97.9, 57.6)
- added C24: 100nF, Capacitor_SMD:C_0805_2012Metric, F.Cu at (102.3, 54.6)
- added C25: 100nF, Capacitor_SMD:C_0805_2012Metric, F.Cu at (106.7, 51.7)
- added C26: 100nF, Capacitor_SMD:C_0805_2012Metric, F.Cu at (97.9, 60.5)
- added C27: 100nF, Capacitor_SMD:C_0805_2012Metric, F.Cu at (102.3, 57.6)
- added C28: C, Capacitor_SMD:C_0805_2012Metric, F.Cu at (111.1, 51.7)
- added C29: 100nF, Capacitor_SMD:C_0805_2012Metric, F.Cu at (97.9, 51.7)
- added C30: 100nF, Capacitor_SMD:C_0805_2012Metric, F.Cu at (102.3, 60.5)
- added C31: 100nF, Capacitor_SMD:C_0805_2012Metric, F.Cu at (106.7, 57.6)
- added C32: 100nF, Capacitor_SMD:C_0805_2012Metric, F.Cu at (111.1, 54.6)
- added C9: 10uF, Capacitor_SMD:C_0805_2012Metric, F.Cu at (90.0, 109.3)
- added JP1: Pines_Bloque_50, ZYNQ_7000:PINES_50, F.Cu at (148.6, 135.9)
- added JP2: Pines_Bloque_50, ZYNQ_7000:PINES_50, F.Cu at (167.6, 54.6)
- added L3: 4.7uH, Inductor_SMD:L_0805_2012Metric, F.Cu at (84.4, 119.8)
- added L4: 4.7uH, Inductor_SMD:L_0805_2012Metric, F.Cu at (89.9, 115.2)
- added Q3: MMBT3904, Package_TO_SOT_SMD:SOT-23, F.Cu at (81.1, 110.1)
- added Q4: MMBT3904, Package_TO_SOT_SMD:SOT-23, F.Cu at (75.6, 118.9)
- added R10: 79k, Resistor_SMD:R_0805_2012Metric, F.Cu at (89.9, 118.2)
- added R11: 100k, Resistor_SMD:R_0805_2012Metric, F.Cu at (80.1, 125.7)
- added R12: 33k, Resistor_SMD:R_0805_2012Metric, F.Cu at (84.5, 131.6)
- added R13: 100k, Resistor_SMD:R_0805_2012Metric, F.Cu at (80.1, 128.6)
- added R14: 100k, Resistor_SMD:R_0805_2012Metric, F.Cu at (98.8, 112.2)
- added R15: 75k, Resistor_SMD:R_0805_2012Metric, F.Cu at (84.5, 125.7)
- added R16: 0R, Resistor_SMD:R_0805_2012Metric, F.Cu at (88.8, 121.1)
- added R17: 0R, Resistor_SMD:R_0805_2012Metric, F.Cu at (80.1, 131.6)
- added R18: 240R 1%, Resistor_SMD:R_0805_2012Metric, F.Cu at (90.8, 100.7)
- added R19: 1k 1%, Resistor_SMD:R_0805_2012Metric, F.Cu at (115.5, 51.7)
- added R20: 1k 1%, Resistor_SMD:R_0805_2012Metric, F.Cu at (106.7, 60.5)
- added R21: 1k 1%, Resistor_SMD:R_0805_2012Metric, F.Cu at (100.3, 71.1)
- added R22: 1k 1%, Resistor_SMD:R_0805_2012Metric, F.Cu at (114.3, 63.5)
- added R8: 33k, Resistor_SMD:R_0805_2012Metric, F.Cu at (98.8, 109.3)
- added R9: 100k, Resistor_SMD:R_0805_2012Metric, F.Cu at (94.3, 118.2)
- added U3: TPS563201, ZYNQ_7000:TPS563201, F.Cu at (76.2, 110.0)
- added U4: TPS563201, ZYNQ_7000:TPS563201, F.Cu at (97.0, 103.2)
- added U5: XC7Z010-BUENO, ZYNQ_7000:BGA-400_20x20_17.0x17.0mm, F.Cu at (116.8, 84.7)
- added U6: MT41K256M16TW-107_P, ZYNQ_7000:BGA-144_9x16_8.0x14.0mm, F.Cu at (92.7, 83.8)
- C2: value 100nF -> 10uF
- C5, C7, C8: value 10uF -> 100nF
- R2: value 33k -> 10k
- R3: value 100k -> 0R
- R6: value 100k -> 10k
- R7: value 75k -> 10k
- moved L2 262.8 mm to (75.7, 128.6)
- moved R2 260.3 mm to (84.4, 122.7)
- moved R1 257.6 mm to (75.7, 131.5), turned to 0 degrees
- moved C6 256.7 mm to (75.5, 122.7)
- moved C7 256.6 mm to (81.1, 116.8)
- moved R4 253.9 mm to (88.9, 124.0)
- moved R6 252.3 mm to (84.5, 128.6)
- moved U1 251.9 mm to (76.2, 114.5)
- moved R3 250.0 mm to (94.4, 112.2)
- moved C5 247.5 mm to (80.0, 122.7)
- moved C8 245.9 mm to (85.5, 113.8)
- moved R5 243.2 mm to (93.2, 121.1)
- moved R7 243.0 mm to (98.7, 115.2)
- moved L1 242.2 mm to (94.4, 109.3)
- moved Q1 241.4 mm to (85.6, 110.1)
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Connections:
- C2 pad 1: Net-(C2-Pad1) -> VCC
- C2 pad 2: Net-(C2-Pad2) -> GND
- C3 pad 1: +1V0 -> VCC
- C4 pad 1: +1V0 -> VCC
- C5 pad 1: VCC -> Net-(C5-Pad1)
- C5 pad 2: GND -> Net-(C5-Pad2)
- C7 pad 1: +1V8 -> Net-(C7-Pad1)
- C7 pad 2: GND -> Net-(C7-Pad2)
- C8 pad 1: +1V8 -> Net-(C8-Pad1)
- C8 pad 2: GND -> Net-(C8-Pad2)
- L1 pad 1: Net-(C2-Pad1) -> Net-(C5-Pad1)
- L1 pad 2: +1V0 -> +1V35
- L2 pad 2: +1V8 -> +1V0
- Q1 pad 1: +1V0 -> Net-(Q1-Pad1)
- Q2 pad 1: Net-(Q1-Pad3) -> +1V0
- R1 pad 1: Net-(R1-Pad1) -> Net-(Q1-Pad1)
- R1 pad 2: VCC -> +1V35
- R2 pad 1: +1V0 -> Net-(Q1-Pad3)
- R2 pad 2: Net-(R2-Pad2) -> VCC
- R3 pad 1: Net-(R2-Pad2) -> Net-(R3-Pad1)
- R3 pad 2: GND -> +1V8
- R4 pad 1: Net-(Q1-Pad3) -> Net-(R4-Pad1)
- R6 pad 1: +1V8 -> Net-(Q3-Pad3)
- R6 pad 2: Net-(R6-Pad2) -> VCC
- R7 pad 1: Net-(R6-Pad2) -> Net-(Q4-Pad3)
- R7 pad 2: GND -> VCC
- U1 pad 2: Net-(C6-Pad1) -> Net-(C5-Pad1)
- U1 pad 4: Net-(R6-Pad2) -> Net-(R10-Pad2)
- U1 pad 5: Net-(Q2-Pad3) -> Net-(R3-Pad1)
- U1 pad 6: Net-(C6-Pad2) -> Net-(C5-Pad2)
- U2 pad 2: Net-(C2-Pad1) -> Net-(C6-Pad1)
- U2 pad 4: Net-(R2-Pad2) -> Net-(R8-Pad2)
- U2 pad 5: Net-(R1-Pad1) -> Net-(R4-Pad1)
- U2 pad 6: Net-(C2-Pad2) -> Net-(C6-Pad2)
