File: Diseno_1/Diseno_1.kicad_pcb (KiCad board)
At the start: 2 copper layers, 70 parts, among them Q1 MMBT3904, Q2 MMBT3904, Q3 MMBT3904, Q4 MMBT3904, U1 TPS563201, U2 TPS563201, U3 TPS563201, U4 TPS563201, U5 XC7Z010-BUENO, U6 MT41K256M16TW-107_P

Commit message: actualizacion
Parts:
- added J1: Conn_01x06, Connector_PinHeader_2.54mm:PinHeader_1x06_P2.54mm_Vertical, F.Cu at (135.9, 40.6)
- moved JP2 20.7 mm to (171.4, 74.9)
Connections:
- U5 pad F6: (no net) -> /Referencias y MIOs/TDO
- U5 pad F9: (no net) -> /Referencias y MIOs/TCK
- U5 pad G6: (no net) -> /Referencias y MIOs/TDI
- U5 pad J6: (no net) -> /Referencias y MIOs/TMS
- U5 pad N6: (no net) -> +3V3
- U5 pad R6: (no net) -> +3V3
- U5 pad T6: (no net) -> +3V3
Other:
- board outline added: 114.3 x 108 mm
- board text added: "3V3"
- board text added: "GND"
- board text added: "JTAG"
- board text added: "TCK"
- board text added: "TDI"
- board text added: "TDO"
- board text added: "TMS"
Changed lines of the file:
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@@
   (general
     (thickness 1.6)
-    (drawings 0)
+    (drawings 11)
     (tracks 0)
     (zones 0)
-    (modules 70)
-    (nets 178)
+    (modules 71)
+    (nets 182)
   )
   (page A3)
@@
     (mod_text_size 1 1)
     (mod_text_width 0.15)
-    (pad_size 1.524 1.524)
-    (pad_drill 0.762)
+    (pad_size 0.5 0.5)
+    (pad_drill 0)
     (pad_to_mask_clearance 0.051)
     (solder_mask_min_width 0.25)
@@
   (net 176 "/Entradas y Salidas/BANK35_C20")
   (net 177 "/Entradas y Salidas/BANK35_G14")
+  (net 178 "/Referencias y MIOs/TMS")
+  (net 179 "/Referencias y MIOs/TDI")
+  (net 180 "/Referencias y MIOs/TDO")
+  (net 181 "/Referencias y MIOs/TCK")
   (net_class Default "Esta es la clase de red por defecto."
     (clearance 0.2)
@@
     (add_net "/Memoria RAM/DDR_VREF")
     (add_net "/Memoria RAM/DDR_WE")
+    (add_net "/Referencias y MIOs/TCK")
+    (add_net "/Referencias y MIOs/TDI")
+    (add_net "/Referencias y MIOs/TDO")
+    (add_net "/Referencias y MIOs/TMS")
     (add_net GND)
     (add_net "Net-(C18-Pad1)")
@@
     (add_net "Net-(U5-PadF14)")
     (add_net "Net-(U5-PadF15)")
-    (add_net "Net-(U5-PadF6)")
-    (add_net "Net-(U5-PadF9)")
-    (add_net "Net-(U5-PadG6)")
-    (add_net "Net-(U5-PadJ6)")
     (add_net "Net-(U5-PadL6)")
     (add_net "Net-(U5-PadM6)")
     (add_net "Net-(U5-PadN5)")
-    (add_net "Net-(U5-PadN6)")
     (add_net "Net-(U5-PadP1)")
     (add_net "Net-(U5-PadP3)")
@@
     (add_net "Net-(U5-PadR2)")
     (add_net "Net-(U5-PadR3)")
-    (add_net "Net-(U5-PadR6)")
     (add_net "Net-(U5-PadT1)")
     (add_net "Net-(U5-PadT2)")
     (add_net "Net-(U5-PadT4)")
     (add_net "Net-(U5-PadT5)")
-    (add_net "Net-(U5-PadT6)")
     (add_net "Net-(U5-PadT9)")
     (add_net "Net-(U5-PadU10)")
@@
     (add_net VCC)
   )
+  (module Connector_PinHeader_2.54mm:PinHeader_1x06_P2.54mm_Vertical (layer F.Cu)
+    (at 135.89 40.64)
+    (descr "Through hole straight pin header, 1x06, 2.54mm pitch, single row")
+    (tags "Through hole pin header THT 1x06 2.54mm single row")
+    (fp_text reference J1 (at 0 -2.33) (layer F.SilkS)
+      (effects (font (size 1 1) (thickness 0.15)))
+    )
+    (fp_text value Conn_01x06 (at 0 15.03) (layer F.Fab)
+      (effects (font (size 1 1) (thickness 0.15)))
+    )
+    (fp_text user %R (at 0 6.35 90) (layer F.Fab)
+      (effects (font (size 1 1) (thickness 0.15)))
+    )
+    (fp_line (start 1.8 -1.8) (end -1.8 -1.8) (layer F.CrtYd) (width 0.05))
+    (fp_line (start 1.8 14.5) (end 1.8 -1.8) (layer F.CrtYd) (width 0.05))
+    (fp_line (start -1.8 14.5) (end 1.8 14.5) (layer F.CrtYd) (width 0.05))
+    (fp_line (start -1.8 -1.8) (end -1.8 14.5) (layer F.CrtYd) (width 0.05))
+    (fp_line (start -1.33 -1.33) (end 0 -1.33) (layer F.SilkS) (width 0.12))
+    (fp_line (start -1.33 0) (end -1.33 -1.33) (layer F.SilkS) (width 0.12))
+    (fp_line (start -1.33 1.27) (end 1.33 1.27) (layer F.SilkS) (width 0.12))
+    (fp_line (start 1.33 1.27) (end 1.33 14.03) (layer F.SilkS) (width 0.12))
+    (fp_line (start -1.33 1.27) (end -1.33 14.03) (layer F.SilkS) (width 0.12))
+    (fp_line (start -1.33 14.03) (end 1.33 14.03) (layer F.SilkS) (width 0.12))
+    (fp_line (start -1.27 -0.635) (end -0.635 -1.27) (layer F.Fab) (width 0.1))
+    (fp_line (start -1.27 13.97) (end -1.27 -0.635) (layer F.Fab) (width 0.1))
+    (fp_line (start 1.27 13.97) (end -1.27 13.97) (layer F.Fab) (width 0.1))
+    (fp_line (start 1.27 -1.27) (end 1.27 13.97) (layer F.Fab) (width 0.1))
+    (fp_line (start -0.635 -1.27) (end 1.27 -1.27) (layer F.Fab) (width 0.1))
+    (pad 6 thru_hole oval (at 0 12.7) (size 1.7 1.7) (drill 1) (layers *.Cu *.Mask)
+      (net 178 "/Referencias y MIOs/TMS"))
+    (pad 5 thru_hole oval (at 0 10.16) (size 1.7 1.7) (drill 1) (layers *.Cu *.Mask)
+      (net 179 "/Referencias y MIOs/TDI"))
+    (pad 4 thru_hole oval (at 0 7.62) (size 1.7 1.7) (drill 1) (layers *.Cu *.Mask)
+      (net 180 "/Referencias y MIOs/TDO"))
+    (pad 3 thru_hole oval (at 0 5.08) (size 1.7 1.7) (drill 1) (layers *.Cu *.Mask)
+      (net 181 "/Referencias y MIOs/TCK"))
+    (pad 2 thru_hole oval (at 0 2.54) (size 1.7 1.7) (drill 1) (layers *.Cu *.Mask)
+      (net 1 GND))
+    (pad 1 thru_hole rect (at 0 0) (size 1.7 1.7) (drill 1) (layers *.Cu *.Mask)
+      (net 13 +3V3))
+    (model ${KISYS3DMOD}/Connector_PinHeader_2.54mm.3dshapes/PinHeader_1x06_P2.54mm_Vertical.wrl
+      (at (xyz 0 0 0))
+      (scale (xyz 1 1 1))
+      (rotate (xyz 0 0 0))
+    )
+  )
   (module ZYNQ_7000:PINES_50 (layer F.Cu)
-    (at 167.64 54.61 180)
+    (at 171.45 74.93 180)
     (fp_text reference JP2 (at -1.143 33.909) (layer F.SilkS)
       (effects (font (size 1 1) (thickness 0.15)))
@@
     (pad G9 smd circle (at -1.2 -2.8) (size 0.5 0.5) (layers F.Cu F.Paste F.Mask)
       (net 14 +1V8))
-    (pad F9 smd circle (at -1.2 -3.6) (size 0.5 0.5) (layers F.Cu F.Paste F.Mask))
+    (pad F9 smd circle (at -1.2 -3.6) (size 0.5 0.5) (layers F.Cu F.Paste F.Mask)
+      (net 181 "/Referencias y MIOs/TCK"))
     (pad E9 smd circle (at -1.2 -4.4) (size 0.5 0.5) (layers F.Cu F.Paste F.Mask))
     (pad D9 smd circle (at -1.2 -5.2) (size 0.5 0.5) (layers F.Cu F.Paste F.Mask))
@@
     (pad U6 smd circle (at -3.6 5.2) (size 0.5 0.5) (layers F.Cu F.Paste F.Mask)
       (net 1 GND))
-    (pad T6 smd circle (at -3.6 4.4) (size 0.5 0.5) (layers F.Cu F.Paste F.Mask))
-    (pad R6 smd circle (at -3.6 3.6) (size 0.5 0.5) (layers F.Cu F.Paste F.Mask))
+    (pad T6 smd circle (at -3.6 4.4) (size 0.5 0.5) (layers F.Cu F.Paste F.Mask)
+      (net 13 +3V3))
+    (pad R6 smd circle (at -3.6 3.6) (size 0.5 0.5) (layers F.Cu F.Paste F.Mask)
+      (net 13 +3V3))
     (pad P6 smd circle (at -3.6 2.8) (size 0.5 0.5) (layers F.Cu F.Paste F.Mask)
       (net 26 "/Memoria RAM/DDR_VREF"))
-    (pad N6 smd circle (at -3.6 2) (size 0.5 0.5) (layers F.Cu F.Paste F.Mask))
+    (pad N6 smd circle (at -3.6 2) (size 0.5 0.5) (layers F.Cu F.Paste F.Mask)
+      (net 13 +3V3))
     (pad M6 smd circle (at -3.6 1.2) (size 0.5 0.5) (layers F.Cu F.Paste F.Mask))
     (pad L6 smd circle (at -3.6 0.4) (size 0.5 0.5) (layers F.Cu F.Paste F.Mask))
     (pad K6 smd circle (at -3.6 -0.4) (size 0.5 0.5) (layers F.Cu F.Paste F.Mask)
       (net 13 +3V3))
-    (pad J6 smd circle (at -3.6 -1.2) (size 0.5 0.5) (layers F.Cu F.Paste F.Mask))
+    (pad J6 smd circle (at -3.6 -1.2) (size 0.5 0.5) (layers F.Cu F.Paste F.Mask)
+      (net 178 "/Referencias y MIOs/TMS"))
     (pad H6 smd circle (at -3.6 -2) (size 0.5 0.5) (layers F.Cu F.Paste F.Mask)
       (net 26 "/Memoria RAM/DDR_VREF"))
-    (pad G6 smd circle (at -3.6 -2.8) (size 0.5 0.5) (layers F.Cu F.Paste F.Mask))
-    (pad F6 smd circle (at -3.6 -3.6) (size 0.5 0.5) (layers F.Cu F.Paste F.Mask))
+    (pad G6 smd circle (at -3.6 -2.8) (size 0.5 0.5) (layers F.Cu F.Paste F.Mask)
+      (net 179 "/Referencias y MIOs/TDI"))
+    (pad F6 smd circle (at -3.6 -3.6) (size 0.5 0.5) (layers F.Cu F.Paste F.Mask)
+      (net 180 "/Referencias y MIOs/TDO"))
     (pad E6 smd circle (at -3.6 -4.4) (size 0.5 0.5) (layers F.Cu F.Paste F.Mask))
     (pad D6 smd circle (at -3.6 -5.2) (size 0.5 0.5) (layers F.Cu F.Paste F.Mask))
@@
   (module ZYNQ_7000:TPS563201 (layer F.Cu)
     (at 76.181 110.036)
-    (fp_text reference U3 (at -0.508 -2.921) (layer F.SilkS)
+    (fp_text reference U3 (at -3.791 0.454 90) (layer F.SilkS)
       (effects (font (size 1 1) (thickness 0.15)))
     )
@@
     )
   )
+  (gr_text JTAG (at 135.89 57.15) (layer F.SilkS)
+    (effects (font (size 1 1) (thickness 0.15)))
+  )
+  (gr_text TDI (at 139.7 50.8) (layer F.SilkS)
+    (effects (font (size 1 1) (thickness 0.15)))
+  )
+  (gr_text TMS (at 139.7 53.34) (layer F.SilkS)
+    (effects (font (size 1 1) (thickness 0.15)))
+  )
+  (gr_text "TDO\n" (at 139.7 48.26) (layer F.SilkS)
+    (effects (font (size 1 1) (thickness 0.15)))
+  )
+  (gr_text TCK (at 139.7 45.72) (layer F.SilkS)
+    (effects (font (size 1 1) (thickness 0.15)))
+  )
+  (gr_text GND (at 139.7 43.18) (layer F.SilkS)
+    (effects (font (size 1 1) (thickness 0.15)))
+  )
+  (gr_text 3V3 (at 139.7 40.64) (layer F.SilkS)
+    (effects (font (size 1 1) (thickness 0.15)))
+  )
+  (gr_line (start 182.88 34.29) (end 68.58 34.29) (layer Edge.Cuts) (width 0.05))
+  (gr_line (start 182.88 142.24) (end 182.88 34.29) (layer Edge.Cuts) (width 0.05))
+  (gr_line (start 68.58 142.24) (end 182.88 142.24) (layer Edge.Cuts) (width 0.05))
+  (gr_line (start 68.58 142.24) (end 68.58 34.29) (layer Edge.Cuts) (width 0.05))
 )

Commit message: actualizacion
Parts:
- added C33: 100nF, Capacitor_SMD:C_0805_2012Metric, F.Cu at (153.7, 91.4)
- added C34: 100nF, Capacitor_SMD:C_0805_2012Metric, F.Cu at (158.1, 91.4)
- added R23: 240R 1%, Resistor_SMD:R_0805_2012Metric, F.Cu at (153.7, 94.4)
- added SW1: SW_Push, Button_Switch_SMD:SW_SPST_CK_RS282G05A3, F.Cu at (203.2, 100.3)
- added U7: MT41K256M16TW-107_P, ZYNQ_7000:BGA-144_9x16_8.0x14.0mm, F.Cu at (171.4, 105.4)
- moved Q4 128.4 mm to (202.3, 139.5)
- moved L3 128.4 mm to (211.1, 140.3)
- moved R1 128.4 mm to (202.4, 152.1)
- moved R12 128.4 mm to (211.2, 152.1)
- moved R13 128.4 mm to (206.8, 149.2)
- moved R15 128.4 mm to (211.2, 146.2)
- moved R17 128.4 mm to (206.8, 152.1)
- moved R2 128.4 mm to (211.1, 143.3)
- moved R6 128.4 mm to (211.2, 149.2)
- moved C11 112.3 mm to (176.0, 175.8)
- moved U1 109.8 mm to (169.4, 172.5)
- moved C13 105.2 mm to (186.5, 154.2)
- moved C15 105.2 mm to (177.6, 155.8)
- moved C7 105.2 mm to (177.6, 158.7)
- moved Q1 105.2 mm to (182.1, 152.0)
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Connections:
- JP1 pad 11: /Entradas y Salidas/BANK34_U13 -> (no net)
- U5 pad N5: (no net) -> /Memoria RAM/DDR_ODT
- U5 pad P1: (no net) -> /Memoria RAM/DDR_D16
- U5 pad P3: (no net) -> /Memoria RAM/DDR_D17
- U5 pad R1: (no net) -> /Memoria RAM/DDR_D19
- U5 pad R2: (no net) -> /Memoria RAM/DDR_DQS2+
- U5 pad R3: (no net) -> /Memoria RAM/DDR_D18
- U5 pad T1: (no net) -> /Memoria RAM/DDR_DQM2
- U5 pad T2: (no net) -> /Memoria RAM/DDR_DQS2-
- U5 pad T4: (no net) -> /Memoria RAM/DDR_D20
- U5 pad U13: /Entradas y Salidas/BANK34_U13 -> GND
- U5 pad U2: (no net) -> /Memoria RAM/DDR_D22
- U5 pad U3: (no net) -> /Memoria RAM/DDR_D23
- U5 pad U4: (no net) -> /Memoria RAM/DDR_D21
- U5 pad V1: (no net) -> /Memoria RAM/DDR_D24
- U5 pad V2: (no net) -> /Memoria RAM/DDR_D30
- U5 pad V3: (no net) -> /Memoria RAM/DDR_D31
- U5 pad W1: (no net) -> /Memoria RAM/DDR_D26
- U5 pad W3: (no net) -> /Memoria RAM/DDR_D29
- U5 pad W4: (no net) -> /Memoria RAM/DDR_DQS3-
- U5 pad W5: (no net) -> /Memoria RAM/DDR_DQS3+
- U5 pad Y1: (no net) -> /Memoria RAM/DDR_DQM3
- U5 pad Y2: (no net) -> /Memoria RAM/DDR_D28
- U5 pad Y3: (no net) -> /Memoria RAM/DDR_D25
- U5 pad Y4: (no net) -> /Memoria RAM/DDR_D27
- U6 pad K1: (no net) -> /Memoria RAM/DDR_ODT
- U6 pad L3: (no net) -> /Memoria RAM/DDR_WE
Routing:
- net /Referencias y MIOs/TMS: track 0.00 -> 71.2 mm, vias 0 -> 1
- net /Referencias y MIOs/TCK: track 0.00 -> 62.7 mm, vias 0 -> 1
- net /Referencias y MIOs/TDI: track 0.00 -> 61.9 mm, vias 0 -> 3
- net /Referencias y MIOs/TDO: track 0.00 -> 60.5 mm, vias 0 -> 2
- net Net-(C5-Pad1): track 0.00 -> 20.0 mm, vias 0 -> 3
- net GND: track 0.00 -> 13.0 mm, vias 0 -> 7
- net +1V0: track 0.00 -> 12.5 mm
- net Net-(C6-Pad1): track 0.00 -> 12.1 mm, vias 0 -> 2
- net Net-(R8-Pad2): track 0.00 -> 10.6 mm, vias 0 -> 2
- net +1V35: track 0.00 -> 8.76 mm
- net Net-(R3-Pad1): track 0.00 -> 5.38 mm
- net VCC: track 0.00 -> 5.14 mm
- net Net-(R4-Pad1): track 0.00 -> 4.96 mm
- net Net-(R10-Pad2): track 0.00 -> 4.50 mm
- net Net-(C5-Pad2): track 0.00 -> 4.17 mm
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Other:
- board size 114.3 x 108 mm -> 82.6 x 108 mm

Commit message: ACT
Parts:
- added C35: 4.7uF, Resistor_SMD:R_0805_2012Metric, F.Cu at (214.0, 169.2)
- added C36: 100nF, Resistor_SMD:R_0805_2012Metric, F.Cu at (216.2, 159.0)
- added J2: USB_B_Micro, Connector_USB:USB_Mini-B_Lumberg_2486_01_Horizontal, F.Cu at (210.3, 175.6)
- added R24: 4.7k, Resistor_SMD:R_0805_2012Metric, F.Cu at (217.3, 169.2)
- added R25: 10k, Resistor_SMD:R_0805_2012Metric, F.Cu at (214.1, 164.5)
- added R26: 1k, Resistor_SMD:R_0805_2012Metric, F.Cu at (217.2, 162.7)
- added R27: 4.7K, Resistor_SMD:R_0805_2012Metric, F.Cu at (161.1, 127.1)
- added R28: 4.7K, Resistor_SMD:R_0805_2012Metric, F.Cu at (164.1, 122.4)
- added U8: CP2102N-A01-GQFN28, Package_DFN_QFN:QFN-28-1EP_5x5mm_P0.5mm_EP3.35x3.35mm, F.Cu at (209.1, 164.0)
- JP1, JP2: footprint ZYNQ_7000:PINES_50 -> ZYNQ_7000:PINES_50_NUMERO
- moved R12 6.23 mm to (206.8, 147.7)
- moved R13 6.23 mm to (202.4, 144.8)
- moved R15 6.23 mm to (206.8, 141.8)
- moved R17 6.23 mm to (202.4, 147.7)
- moved R2 6.23 mm to (206.7, 138.9)
- moved R6 6.23 mm to (206.8, 144.8)
- moved L3 6.23 mm to (206.7, 135.9)
- moved JP2 3.37 mm to (216.9, 121.5), turned to 0 degrees
- moved JP1 2.52 mm to (145.4, 122.8), turned to 0 degrees
Connections:
- U5 pad A16: (no net) -> /Referencias y MIOs/MIO24
- U5 pad F15: (no net) -> /Referencias y MIOs/MIO25
- U5 pad J9: GND -> +1V8
- U5 pad L6: (no net) -> Net-(R28-Pad2)
- U5 pad M6: (no net) -> +3V3
- U5 pad R10: (no net) -> Net-(R27-Pad2)
Routing:
- net Net-(C36-Pad2): track 0.00 -> 19.0 mm, vias 0 -> 2
- net Net-(C35-Pad2): track 0.00 -> 16.4 mm
- net Net-(R24-Pad2): track 0.00 -> 7.56 mm
- net Net-(J2-Pad2): track 0.00 -> 6.89 mm, vias 0 -> 2
- net (no net): track 0.00 -> 4.20 mm, vias 0 -> 1
- net Net-(J2-Pad3): track 0.00 -> 3.99 mm, vias 0 -> 1
- net GND: track 13.0 -> 15.7 mm, vias 7 -> 8

Commit message: muchas cosas
Parts:
- added C37: 100nF, Capacitor_SMD:C_0805_2012Metric, F.Cu at (242.6, 161.9)
- added J3: Micro_SD_Card, Connector_Card:microSD_HC_Wuerth_693072010801, F.Cu at (197.8, 197.2)
- added R29: 4.7k, Resistor_SMD:R_0805_2012Metric, F.Cu at (239.4, 161.9)
- added X1: SG-8002JC, Oscillator:Oscillator_SMD_SeikoEpson_SG8002JC-4Pin_10.5x5.0mm, F.Cu at (231.1, 161.9)
- C28: value C -> 100nF
- moved JP2 63.9 mm to (280.0, 130.8)
- moved U8 44.1 mm to (247.6, 185.5)
- moved C36 44.1 mm to (254.7, 180.5)
- moved R25 44.1 mm to (252.5, 186.1)
- moved R26 44.1 mm to (255.7, 184.3)
- moved R24 44.1 mm to (255.7, 190.7)
- moved C35 44.1 mm to (252.4, 190.8)
- moved J2 44.1 mm to (248.8, 197.1)
Connections:
- U5 pad A9: (no net) -> /Referencias y MIOs/SD_D1
- U5 pad B15: (no net) -> /Referencias y MIOs/SD_D3
- U5 pad C17: (no net) -> /Referencias y MIOs/SD_CMD
- U5 pad D14: (no net) -> /Referencias y MIOs/SD_CLK
- U5 pad E12: (no net) -> /Referencias y MIOs/SD_D0
- U5 pad E7: (no net) -> /Referencias y MIOs/PS_CLK
- U5 pad F13: (no net) -> /Referencias y MIOs/SD_D2
Routing:
- net +3V3: track 0.00 -> 10.0 mm
- net Net-(R29-Pad2): track 0.00 -> 6.85 mm
Other:
- board size 82.6 x 108 mm -> 146.1 x 129.5 mm
