File: Diseno_1/alimentaciones.sch (KiCad schematic (older format))
At the start: 46 parts, among them Q1 MMBT3904, Q2 MMBT3904, Q3 MMBT3904, Q4 MMBT3904, U1 TPS563201, U2 TPS563201, U3 TPS563201, U4 TPS563201, U5 XC7Z010-BUENO

Commit message: muchas cosas
Other:
- note added: "VIN -> 1V0, 1V8, 3V3 & 1V35 \n"
- note added: "XC7Z010\n"
- moved on the sheet: U?H, U?I
