File: Diseno_1/referencia.sch (KiCad schematic (older format))
At the start: 1 part, among them U5 XC7Z010-BUENO

Commit message: actualizacion
Parts:
- added J1: Conn_01x06, Connector_PinHeader_2.54mm:PinHeader_1x06_P2.54mm_Vertical, symbol Connector_Generic:Conn_01x06
Connections:
- net +3V3: now also J1.1 (Pin_1)
- net GND: now also J1.2 (Pin_2)
- net TDO: now reaches U5.F6 (TDO_0)
- net TDO: now also J1.4 (Pin_4)
- net TCK: now reaches U5.F9 (TCK_0)
- net TCK: now also J1.3 (Pin_3)
- net TDI: now reaches U5.G6 (TDI_0)
- net TDI: now also J1.5 (Pin_5)
- net TMS: now reaches U5.J6 (TMS_0)
- net TMS: now also J1.6 (Pin_6)
- no-connect marks 0 -> 1
Changed lines of the file:
@@
 	13200 8550 12950 8550
 Connection ~ 13200 8450
+$Comp
+L Connector_Generic:Conn_01x06 J1
+U 1 1 5FF10D81
+P 2100 3900
+F 0 "J1" H 2018 3375 50  0000 C CNN
+F 1 "Conn_01x06" H 2018 3466 50  0000 C CNN
+F 2 "Connector_PinHeader_2.54mm:PinHeader_1x06_P2.54mm_Vertical" H 2100 3900 50  0001 C CNN
+F 3 "~" H 2100 3900 50  0001 C CNN
+	1    2100 3900
+	-1   0    0    -1
+$EndComp
+Text Label 2550 3900 2    50   ~ 0
+TCK
+Text Label 2550 4000 2    50   ~ 0
+TDO
+Text Label 2550 4100 2    50   ~ 0
+TDI
+Text Label 2550 4200 2    50   ~ 0
+TMS
+Wire Wire Line
+	2550 3900 2300 3900
+Wire Wire Line
+	2300 4000 2550 4000
+Wire Wire Line
+	2550 4100 2300 4100
+Wire Wire Line
+	2300 4200 2550 4200
+$Comp
+L power:GND #PWR0120
+U 1 1 5FF1E8BE
+P 2650 3800
+F 0 "#PWR0120" H 2650 3550 50  0001 C CNN
+F 1 "GND" V 2655 3672 50  0000 R CNN
+F 2 "" H 2650 3800 50  0001 C CNN
+F 3 "" H 2650 3800 50  0001 C CNN
+	1    2650 3800
+	0    -1   -1   0
+$EndComp
+Wire Wire Line
+	2650 3800 2300 3800
+$Comp
+L power:+3.3V #PWR0121
+U 1 1 5FF20956
+P 2550 3600
+F 0 "#PWR0121" H 2550 3450 50  0001 C CNN
+F 1 "+3.3V" H 2565 3773 50  0000 C CNN
+F 2 "" H 2550 3600 50  0001 C CNN
+F 3 "" H 2550 3600 50  0001 C CNN
+	1    2550 3600
+	1    0    0    -1
+$EndComp
+Wire Wire Line
+	2550 3700 2300 3700
+Wire Wire Line
+	2550 3600 2550 3700
+Text Label 13250 7400 2    50   ~ 0
+TMS
+Text Label 13250 7500 2    50   ~ 0
+TCK
+Text Label 13250 7600 2    50   ~ 0
+TDI
+Text Label 13250 7700 2    50   ~ 0
+TDO
+Wire Wire Line
+	13250 7700 12950 7700
+Wire Wire Line
+	12950 7600 13250 7600
+Wire Wire Line
+	13250 7500 12950 7500
+Wire Wire Line
+	12950 7400 13250 7400
+NoConn ~ 8150 5350
 $EndSCHEMATC

Commit message: actualizacion
Parts:
- added SW1: SW_Push, Button_Switch_SMD:SW_SPST_CK_RS282G05A3, symbol Switch:SW_Push
Changed lines of the file:
@@
 Wire Wire Line
 	2300 4000 2550 4000
-Wire Wire Line
-	2550 4100 2300 4100
-Wire Wire Line
-	2300 4200 2550 4200
 $Comp
 L power:GND #PWR0120
@@
 	12950 7400 13250 7400
 NoConn ~ 8150 5350
+$Comp
+L Switch:SW_Push SW1
+U 1 1 5FF49A4D
+P 4900 7600
+F 0 "SW1" H 4900 7885 50  0000 C CNN
+F 1 "SW_Push" H 4900 7794 50  0000 C CNN
+F 2 "Button_Switch_SMD:SW_SPST_CK_RS282G05A3" H 4900 7800 50  0001 C CNN
+F 3 "~" H 4900 7800 50  0001 C CNN
+	1    4900 7600
+	1    0    0    -1
+$EndComp
+Wire Wire Line
+	2300 4100 3800 4100
+Wire Wire Line
+	2300 4200 4200 4200
 $EndSCHEMATC

Commit message: ACT
Parts:
- added C35: 4.7uF, Resistor_SMD:R_0805_2012Metric, symbol Device:C
- added C36: 100nF, Resistor_SMD:R_0805_2012Metric, symbol Device:C
- added J2: USB_B_Micro, Connector_USB:USB_Mini-B_Lumberg_2486_01_Horizontal, symbol Connector:USB_B_Micro
- added R24: 4.7k, Resistor_SMD:R_0805_2012Metric, symbol Device:R
- added R25: 10k, Resistor_SMD:R_0805_2012Metric, symbol Device:R
- added R26: 1k, Resistor_SMD:R_0805_2012Metric, symbol Device:R
- added R27, R28: 4.7K, Resistor_SMD:R_0805_2012Metric, symbol Device:R
- added U8: CP2102N-A01-GQFN28, Package_DFN_QFN:QFN-28-1EP_5x5mm_P0.5mm_EP3.35x3.35mm, symbol Interface_USB:CP2102N-A01-GQFN28
Connections:
- net labels added: +1V8, FPGA_DONE, MIO24, MIO25
- wire segments 35 -> 76
- no-connect marks 1 -> 20
Other:
- moved on the sheet: SW1

Commit message: muchas cosas
Parts:
- removed SW1: SW_Push, Button_Switch_SMD:SW_SPST_CK_RS282G05A3, symbol Switch:SW_Push
- added C37: 100nF, Capacitor_SMD:C_0805_2012Metric, symbol Device:C
- added C? (x2): 27pF, Capacitor_SMD:C_0805_2012Metric, symbol Device:C
- added J3: Micro_SD_Card, Connector_Card:microSD_HC_Wuerth_693072010801, symbol Connector:Micro_SD_Card
- added J?: USB_B_Micro, Connector_USB:USB_Mini-B_Lumberg_2486_01_Horizontal, symbol Connector:USB_B_Micro
- added R29: 4.7k, Resistor_SMD:R_0805_2012Metric, symbol Device:R
- added U?: FT2232H, Package_QFP:LQFP-64-1EP_10x10mm_P0.5mm_EP6.5x6.5mm, symbol Interface_USB:FT2232H
- added U?: 93AAxxB, symbol Memory_EEPROM:93AAxxB
- added X1: SG-8002JC, Oscillator:Oscillator_SMD_SeikoEpson_SG8002JC-4Pin_10.5x5.0mm, symbol Oscillator:SG-8002JC
- added Y?: Crystal, Crystal:Crystal_SMD_0603-2Pin_6.0x3.5mm, symbol Device:Crystal
Connections:
- net +3V3: now also C37.2, J3.4 (VDD), R29.1, X1.4 (V+)
- net GND: now also C37.1, C?.2, C?.2, J3.6 (VSS), J3.9 (SHIELD), J?.5 (GND), J?.6 (Shield), U?.1 (GND), U?.10 (AGND), U?.11 (GND), U?.13 (TEST), U?.15 (GND), U?.25 (GND), U?.35 (GND), U?.47 (GND), U?.5 (GND), U?.5 (GND), U?.51 (GND), X1.2 (GND)
- net TCK: now also U?.16 (ADBUS0)
- net TDI: now also U?.17 (ADBUS1)
- net TDO: now also U?.18 (ADBUS2)
- net TMS: now also U?.19 (ADBUS3)
- net PS_CLK: now reaches U5.E7 (PS_CLK_500)
- net PS_CLK: now also X1.3 (OUT)
- net SD_D1: now reaches U5.A9 (PS_MIO43_501)
- net SD_D1: now also J3.8 (DAT1)
- net SD_D3: now reaches U5.B15 (PS_MIO45_501)
- net SD_D3: now also J3.2 (DAT3/CD)
- net SD_CMD: now reaches U5.C17 (PS_MIO41_501)
- net SD_CMD: now also J3.3 (CMD)
- net SD_CLK: now reaches U5.D14 (PS_MIO40_501)
- net SD_CLK: now also J3.5 (CLK)
- net SD_D0: now reaches U5.E12 (PS_MIO42_501)
- net SD_D0: now also J3.7 (DAT0)
- net SD_D2: now reaches U5.F13 (PS_MIO44_501)
- net SD_D2: now also J3.1 (DAT2)
- new net: R29.2, X1.1 (OE)
- new net: C?.1, U?.2 (OSCI), Y?.1
- new net: C?.1, U?.3 (OSCO), Y?.2
- new net: J?.2 (D-), U?.7 (DM)
- new net: J?.3 (D+), U?.8 (DP)
- new net EECLK: U?.2 (SCLK), U?.62 (EECLK)
- new net EECS: U?.1 (CS), U?.63 (EECS)
- new net EEDATA: U?.3 (DI), U?.61 (EEDATA)
- no-connect marks 20 -> 51
Other:
- note added: "JTAG (2 Options: FT2232H and/or pins)"
- note added: "JTAG pins"
- note added: "Oscillator 33MHz\n"
- note added: "SD Connector (MIO 40-45)\n"
- note added: "UART (MIO 25(RX) & MIO24(TX))"
- moved on the sheet: C35, C36, J1, J2, R24, R25, R26, R27, R28, U5A, U5B, U5F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
